Commit message: renaming complete, compiles

File: realsense2_framos_description/urdf/_d415.urdf.xacro (robot description, xacro)
@@ -8,5 +8,5 @@
 <robot name="sensor_d415" xmlns:xacro="http://ros.org/wiki/xacro">
   <!-- Includes -->
-  <xacro:include filename="$(find realsense2_description)/urdf/_materials.urdf.xacro" />
+  <xacro:include filename="$(find realsense2_framos_description)/urdf/_materials.urdf.xacro" />
   <xacro:macro name="sensor_d415" params="parent *origin  name:=camera  use_nominal_extrinsics:=false">
     <xacro:property name="M_PI" value="3.1415926535897931" />
@@ -45,5 +45,5 @@
         <geometry>
           <!-- <box size="${d415_cam_width} ${d415_cam_height} ${d415_cam_depth}"/> -->
-	         <mesh filename="package://realsense2_description/meshes/d415.stl" />
+	         <mesh filename="package://realsense2_framos_description/meshes/d415.stl" />
         </geometry>
         <material name="aluminum"/>

File: realsense2_framos_description/urdf/_d435.urdf.xacro (robot description, xacro)
@@ -8,5 +8,5 @@
 <robot name="sensor_d435" xmlns:xacro="http://ros.org/wiki/xacro">
   <!-- Includes -->
-  <xacro:include filename="$(find realsense2_description)/urdf/_materials.urdf.xacro" />
+  <xacro:include filename="$(find realsense2_framos_description)/urdf/_materials.urdf.xacro" />
   <xacro:macro name="sensor_d435" params="parent *origin name:=camera use_nominal_extrinsics:=false">
     <xacro:property name="M_PI" value="3.1415926535897931" />
@@ -45,5 +45,5 @@
         <geometry>
           <!-- <box size="${d435_cam_width} ${d435_cam_height} ${d435_cam_depth}"/> -->
-	        <mesh filename="package://realsense2_description/meshes/d435.dae" />
+	        <mesh filename="package://realsense2_framos_description/meshes/d435.dae" />
         </geometry>
       </visual>

File: realsense2_framos_description/urdf/_r410.urdf.xacro (robot description, xacro)
@@ -8,5 +8,5 @@
 <robot name="sensor_r410" xmlns:xacro="http://ros.org/wiki/xacro">
   <!-- Includes -->
-  <xacro:include filename="$(find realsense2_description)/urdf/_materials.urdf.xacro" />
+  <xacro:include filename="$(find realsense2_framos_description)/urdf/_materials.urdf.xacro" />
   <xacro:macro name="sensor_r410" params="parent *origin  name:=camera  use_nominal_extrinsics:=false">
     <xacro:property name="M_PI" value="3.1415926535897931" />
@@ -38,5 +38,5 @@
         <geometry>
           <box size="${r410_cam_width} ${r410_cam_height} ${r410_cam_depth}"/>
-          <!--<mesh filename="package://realsense2_description/meshes/r410/r410.dae" />-->
+          <!--<mesh filename="package://realsense2_framos_description/meshes/r410/r410.dae" />-->
         </geometry>
         <material name="aluminum"/>

File: realsense2_framos_description/urdf/_r430.urdf.xacro (robot description, xacro)
@@ -8,5 +8,5 @@
 <robot name="sensor_r430" xmlns:xacro="http://ros.org/wiki/xacro">
   <!-- Includes -->
-  <xacro:include filename="$(find realsense2_description)/urdf/_materials.urdf.xacro" />
+  <xacro:include filename="$(find realsense2_framos_description)/urdf/_materials.urdf.xacro" />
   <xacro:macro name="sensor_r430" params="parent *origin name:=camera use_nominal_extrinsics:=false">
   <xacro:property name="M_PI" value="3.1415926535897931" />
@@ -39,5 +39,5 @@
         <geometry>
           <box size="${r430_cam_width} ${r430_cam_height} ${r430_cam_depth}"/>
-          <!--<mesh filename="package://realsense2_description/meshes/r430/r430.dae" />-->
+          <!--<mesh filename="package://realsense2_framos_description/meshes/r430/r430.dae" />-->
         </geometry>
         <material name="aluminum"/>

File: realsense2_framos_description/urdf/test_d415_camera.urdf.xacro (robot description, xacro)
@@ -1,5 +1,5 @@
 <?xml version="1.0"?>
 <robot name="realsense2_camera" xmlns:xacro="http://ros.org/wiki/xacro">
-  <xacro:include filename="$(find realsense2_description)/urdf/_d415.urdf.xacro" />
+  <xacro:include filename="$(find realsense2_framos_description)/urdf/_d415.urdf.xacro" />
   <link name="base_link" />
   <sensor_d415 parent="base_link">

File: realsense2_framos_description/urdf/test_d435_camera.urdf.xacro (robot description, xacro)
@@ -1,5 +1,5 @@
 <?xml version="1.0"?>
 <robot name="realsense2_camera" xmlns:xacro="http://ros.org/wiki/xacro">
-  <xacro:include filename="$(find realsense2_description)/urdf/_d435.urdf.xacro" />
+  <xacro:include filename="$(find realsense2_framos_description)/urdf/_d435.urdf.xacro" />
   <link name="base_link" />
   <sensor_d435 parent="base_link">

File: realsense2_framos_description/urdf/test_d435_multiple_cameras.urdf.xacro (robot description, xacro)
@@ -1,5 +1,5 @@
 <?xml version="1.0"?>
 <robot name="realsense2_camera" xmlns:xacro="http://ros.org/wiki/xacro">
-  <xacro:include filename="$(find realsense2_description)/urdf/_d435.urdf.xacro" />
+  <xacro:include filename="$(find realsense2_framos_description)/urdf/_d435.urdf.xacro" />
   <link name="base_link" />
   <sensor_d435 parent="base_link" name="camera1">

File: realsense2_framos_description/urdf/test_r410_camera.urdf.xacro (robot description, xacro)
@@ -1,5 +1,5 @@
 <?xml version="1.0"?>
 <robot name="realsense2_camera" xmlns:xacro="http://ros.org/wiki/xacro">
-  <xacro:include filename="$(find realsense2_description)/urdf/_r410.urdf.xacro" />
+  <xacro:include filename="$(find realsense2_framos_description)/urdf/_r410.urdf.xacro" />
   <link name="base_link" />
   <sensor_r410 parent="base_link">

File: realsense2_framos_description/urdf/test_r430_camera.urdf.xacro (robot description, xacro)
@@ -1,5 +1,5 @@
 <?xml version="1.0"?>
 <robot name="realsense2_camera" xmlns:xacro="http://ros.org/wiki/xacro">
-  <xacro:include filename="$(find realsense2_description)/urdf/_r430.urdf.xacro" />
+  <xacro:include filename="$(find realsense2_framos_description)/urdf/_r430.urdf.xacro" />
   <link name="base_link" />
   <sensor_r430 parent="base_link">
